File: V2/Hardware/plant_sensor_v2/plant_sensor_v2.kicad_sch (KiCad schematic)
At the start: 38 parts, among them IC1 ICM-20948, U1 STM32WBA52KGUx, X1 NX1612SA-32.000MHZ-CHP-CIS-3, Y1 Crystal

Commit message: update
Parts:
- removed C21, C22: 56p, symbol Device:C
- removed C23: 1.5p, symbol Device:C
- removed C24: 3.9p, symbol Device:C
- removed C25: 2.7p, symbol Device:C
- removed C7, C8: 100n, symbol Device:C
- removed L3: 1.8n, symbol Device:L
- removed L4: 1.3n, symbol Device:L
- added C26: 100n, symbol Device:C
- added FB1: 47R @ 100Mhz, symbol Device:FerriteBead_Small
- added J1: TC2030_SWD-MCP-NL, sparkfun-nrf52832-breakout:TC2030-MCP-NL, symbol sparkfun-nrf52832-breakout-eagle-import:TC2030_SWD-MCP-NL
- C2: value 100n -> 10µ
- R1: value R -> 10k
Connections:
- net GND: now also J1.5 (GND)
- net CRYSTAL2: now reaches U1.12 (PC15)
- net CRYSTAL2: now also C13.1, Y1.2
- net CRYSTAL1: now reaches U1.13 (PC14)
- net CRYSTAL1: now also C12.1, Y1.1
- net +BATT: now reaches U1.14 (VDD)
- net +BATT: now also C2.1, C3.1, C4.1, C5.1, R1.1, U1.23 (VDD), U1.31 (VDD), C26.1, FB1.2, J1.1 (VCC)
- net SWO: now reaches U1.16 (PB3)
- net SWO: now also J1.6 (SWO/TDO)
- net SWDIO: now reaches U1.19 (PA13)
- net SWDIO: now also J1.2 (SWDIO/TMS)
- net ~{RESET}: now reaches U1.24 (NRST)
- net ~{RESET}: now also R1.2, C26.2, J1.3 (~{RESET})
- net RF: now reaches C18.1, L2.2, U1.25 (RF)
- net OSC_OUT: now reaches U1.28 (OSC_OUT), X1.3
- net OSC_IN: now reaches U1.29 (OSC_IN), X1.1
- net at U1.5 (VDDA): now also C1.1, C6.1, FB1.1
- net at C20.1, L1.1: now also AE1.1 (A)
- removed net +1V8: C1.1, C2.1, C3.1, C4.1, C5.1, C6.1
- new net SWCLK: J1.4 (SWCLK/TCK), U1.18 (PA14)
- now unconnected: U1.17 (PA15)
Other:
- note added: "Debugging"
- note added: "MCU + BLE Long Range 1.71 to 3.6 V max 20mA/GPIO pin"
- note added: "Voltage regulator (not needed?) voltage drop of battery when TX?"
- note removed: "MCU + BLE Long Range 1.71 to 3.6 V"
- note removed: "Voltage regulator"
- company: (none) -> Dramco - KU Leuven
- title: (none) -> Plant Sensor V2
- moved on the sheet: AE1, C1, C12, C13, C14, C15, C16, C17, C18, C19, C20, C3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

Commit message: hardware update
Parts:
- added C21: 22u, symbol Device:C
- added C7: 10u, symbol Device:C
- added C8: 100n, symbol Device:C
- added L3: 2u2, Inductor_SMD:L_Murata_DFE201610P, symbol Device:L
- added R4, R5: R, symbol Device:R
- added U2: TPS63900, Package_SON:WSON-10-1EP_2.5x2.5mm_P0.5mm_EP1.2x2mm_ThermalVias, symbol Regulator_Switching:TPS63900
- C1: value 1µ -> 1u
- C2: value 10µ -> 10u
Connections:
- net +BATT: now also C7.1, U2.1 (EN), U2.10 (VIN), U2.2 (SEL); no longer C2.1, C26.1, C3.1, C4.1, C5.1, FB1.2, J1.1 (VCC), R1.1, U1.14 (VDD), U1.23 (VDD), U1.31 (VDD)
- net GND: now also IC1.11 (FSYNC), IC1.25 (EP), C21.2, C7.2, C8.2, R5.1, U2.11 (GND), U2.3 (CFG1), U2.4 (CFG2), U2.5 (CFG3), U2.8 (GND)
- net MISO: now reaches U1.10 (PB9)
- net MISO: now also IC1.9 (SDO_/_AD0)
- net MOSI: now reaches U1.11 (PB8)
- net MOSI: now also IC1.24 (SDA_/_SDI)
- net ~{SS}: now reaches U1.6 (PA5)
- net ~{SS}: now also IC1.22 (NCS)
- net SCLK: now reaches U1.9 (PA0)
- net SCLK: now also IC1.23 (SCL_/_SCLK)
- net LED: now reaches R2.1
- net IMU_INT: now reaches IC1.12 (INT1)
- new net: C8.1, R4.1, R5.2
- new net: L3.1, U2.7 (LX2)
- new net: L3.2, U2.9 (LX1)
- new net +1V8: C2.1, C21.1, C26.1, C3.1, C4.1, C5.1, FB1.2, J1.1 (VCC), R1.1, U1.14 (VDD), U1.23 (VDD), U1.31 (VDD), U2.6 (VOUT)
- no-connect marks 0 -> 2
Other:
- note added: "81-DFE201612E-2R2MP2"
- note added: "GRM187R60J226ME15"
- note added: "GRM188R61A106ME69"
- note added: "Power from I/O pin? Combining multiple GPIO pins?"
- note added: "SPI"
- note added: "TODO"
- note added: "TPS22960 dual load switch combine LED + battery meas circuit"
- note added: "To calculate"
- note added: "VDD: 1.71 - 3.6V VDDIO: 1.71 - 1.95V Max current: (max) 10mA"
- note removed: "Check pin connections"
- note removed: "Decoupling check datasheet"
- note removed: "I2C or SPI?"
- note removed: "INT?"
- note removed: "Power from I/O pin?"
- note removed: "Voltage regulator (not needed?) voltage drop of battery when TX?"
- moved on the sheet: C10, C11, C12, C13, C2, C26, C9, R1, X1, Y1

Commit message: update hardware
Parts:
- removed L3: 2u2, Inductor_SMD:L_Murata_DFE201610P, symbol Device:L
- removed U2: TPS63900, Package_SON:WSON-10-1EP_2.5x2.5mm_P0.5mm_EP1.2x2mm_ThermalVias, symbol Regulator_Switching:TPS63900
- removed X1: NX1612SA-32.000MHZ-CHP-CIS-3, NX1612SA-32:OSCSC105P160X120X35-4N, symbol NX1612SA-32.000MHZ-CHP-CIS-3:NX1612SA-32.000MHZ-CHP-CIS-3
- added B1: WA-BCMC, Battery_holder:WA-BCMC_79523211, symbol WA-BCMC:WA-BCMC
- added C22: 4.7u, Capacitor_SMD:C_0402_1005Metric, symbol Device:C
- added C23: 10u, Capacitor_SMD:C_0402_1005Metric, symbol Device:C
- added C24, C25: 100n, Capacitor_SMD:C_0402_1005Metric, symbol Device:C
- added L4: 2u2, Inductor_SMD:L_Murata_DFE201610P, symbol Device:L
- added R6: 0, Resistor_SMD:R_0402_1005Metric, symbol Device:R
- added U2: TPS22960RSER, TPS22960:RSE0008A, symbol TPS22960:TPS22960RSER
- added U3: TPS62840DLCR, TPS62840:VSON8_2P1X1P6_TEX, symbol TPS62840:TPS62840DLCR
- added Y2: 32MHz, Crystal:Crystal_SMD_2016-4Pin_2.0x1.6mm, symbol Device:Crystal_GND24
- C1, C10, C11, C15, C16, C18, C19, C20, C26, C3, C4, C5, C6, C9: footprint (none) -> Capacitor_SMD:C_0402_1005Metric
- C12, C13: value x -> 6p; footprint (none) -> Capacitor_SMD:C_0402_1005Metric
- C14, C17, C2: footprint (none) -> Capacitor_SMD:C_0603_1608Metric
- C21: value 22u -> 6p; footprint (none) -> Capacitor_SMD:C_0402_1005Metric
- C7: value 10u -> 6p; footprint (none) -> Capacitor_SMD:C_0402_1005Metric
- C8: value 100n -> 10n; footprint (none) -> Capacitor_SMD:C_0402_1005Metric
- D1: value LED -> LED, RED; footprint (none) -> LED_SMD:LED_0603_1608Metric
- FB1, R1, R2: footprint (none) -> Resistor_SMD:R_0402_1005Metric
- J1: footprint sparkfun-nrf52832-breakout:TC2030-MCP-NL -> Connector:Tag-Connect_TC2030-IDC-NL_2x03_P1.27mm_Vertical
- L1, L2: footprint (none) -> Inductor_SMD:L_0402_1005Metric
- R3: value 10k -> 100k; footprint (none) -> Resistor_SMD:R_0402_1005Metric
- R4: value R -> 470k; footprint (none) -> Resistor_SMD:R_0402_1005Metric
- R5: value R -> 220k; footprint (none) -> Resistor_SMD:R_0402_1005Metric
- Y1: value Crystal -> 32.768kHz; footprint (none) -> Crystal:Crystal_SMD_2012-2Pin_2.0x1.2mm
Connections:
- net +1V8: now also C23.1, C24.1, L4.2, U2.1 (VIN1), U3.8 (VOS); no longer C21.1
- net +BATT: now also B1.1, B1.2, C22.1, C25.1, U2.8 (VIN2), U3.2 (VIN), U3.4 (EN); no longer C7.1
- net GND: now also B1.-, C22.2, C23.2, C24.2, C25.2, R6.2, U2.3 (SR), U2.6 (GND), U3.1 (GND), U3.3 (MODE), U3.6 (STOP), Y2.2, Y2.4
- net IMU_INT: now also U1.8 (PA1)
- net LED: now also U1.21 (PB15)
- net OSC_IN: now also C7.1, Y2.1
- net OSC_OUT: now also C21.1, Y2.3
- net SW_IMU: now reaches C10.1, C11.1, IC1.13 (VDD), IC1.8 (VDDIO)
- net SW_IMU: now also U2.4 (VOUT1)
- net BATT_ADC: now reaches U1.2 (PA8)
- net BATT_ADC: now also C8.1, R4.1, R5.2
- net BATT_EN: now reaches U1.3 (PA7)
- net BATT_EN: now also U2.7 (ON2)
- net IMU_EN: now reaches U1.4 (PA6)
- net IMU_EN: now also U2.2 (ON1)
- net SW_BATT: now reaches R4.2
- net SW_BATT: now also U2.5 (VOUT2)
- new net: L4.1, U3.7 (SW)
- new net: R6.1, U3.5 (VSET)
Other:
- note added: "0 Ohm -> 1V8 0.909k Ohm -> 1V9"
- note added: "Batt: 1.8 - 3.4 V Internal Vref = +-1.2 V Output: 0 - 1.084 V"
- note added: "ECS-.327-12:XTAL ECS-.327-12.5-16-TR"
- note added: "GJM1555C1H6R0CB01"
- note added: "GRM155R60G106ME44D"
- note added: "GRM155R61A475MEAAD"
- note added: "Load Switch"
- note added: "MCU"
- note added: "MLPF-WB-04D3"
- note added: "NX1612SA-32.000MHZ-CHP-CIS-3"
- note added: "Power Supply"
- note removed: "Add 32mhz oscillator"
- note removed: "GRM187R60J226ME15"
- note removed: "GRM188R61A106ME69"
- note removed: "Power from I/O pin? Combining multiple GPIO pins?"
- note removed: "TODO"
- note removed: "TPS22960 dual load switch combine LED + battery meas circuit"
- note removed: "USER LED TODO with MOSFET to VDD RGB LED?"
- moved on the sheet: AE1, C1, C10, C11, C12, C13, C14, C15, C16, C17, C18, C19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

Commit message: update hardware
Parts:
- removed AE1: Antenna_Shield, symbol Device:Antenna_Shield
- removed C18: 1.5p, Capacitor_SMD:C_0402_1005Metric, symbol Device:C
- removed C19: 3.9p, Capacitor_SMD:C_0402_1005Metric, symbol Device:C
- removed C20: 2.7p, Capacitor_SMD:C_0402_1005Metric, symbol Device:C
- removed L1: 1.3n, Inductor_SMD:L_0402_1005Metric, symbol Device:L
- removed L2: 1.8n, Inductor_SMD:L_0402_1005Metric, symbol Device:L
- added E1: 609-2450AT42E0100001, Antenna:XDCR_2450AT42E0100E, symbol 2450AT42E0100E:2450AT42E0100E
- added IC2: MLPF-WB-04D3, MLPF-WB-04D3:BGA6C50P3X2_160X100X68, symbol MLPF-WB-04D3:MLPF-WB-04D3
Connections:
- net GND: now also E1.3, E1.4, IC2.A2 (GND4), IC2.B1 (GND3), IC2.B2 (GND2), IC2.B3 (GND1)
- net RF: now also IC2.A1 (IN)
- new net: E1.1, IC2.A3 (OUT)
Other:
- note added: "609-2450AT42E0100001"
- note added: "RS PRO BATTERY HOLDER, CLIP FOR CR2032 SMT TYPE Stock No: 2378244, 2378245"

Commit message: update hardware
Parts:
- removed C21, C7: 6p, Capacitor_SMD:C_0402_1005Metric, symbol Device:C
- Y1: footprint Crystal:Crystal_SMD_2012-2Pin_2.0x1.2mm -> Crystal3:XTAL_ECS-.327-6-1210-TR
- Y2: footprint Crystal:Crystal_SMD_2016-4Pin_2.0x1.6mm -> Crystal2:OSCSC105P160X120X35-4N
Other:
- note added: "520-.327-6-1210-TR"
- note added: "Caps needed?"
- note added: "Set pins to analog mode for lowest power consumption"
- note added: "Vin: 1V8 - 6V5"
- note added: "needed?"
- note removed: "ECS-.327-12:XTAL ECS-.327-12.5-16-TR"

Commit message: hardware update
Parts:
- removed C14: 470n, Capacitor_SMD:C_0603_1608Metric, symbol Device:C
- removed C16, C3, C4, C5, C6: 100n, Capacitor_SMD:C_0402_1005Metric, symbol Device:C
- removed C17: 4.7µ, Capacitor_SMD:C_0603_1608Metric, symbol Device:C
- removed C8: 10n, Capacitor_SMD:C_0402_1005Metric, symbol Device:C
- removed FB1: 47R @ 100Mhz, Resistor_SMD:R_0402_1005Metric, symbol Device:FerriteBead_Small
- removed IC2: MLPF-WB-04D3, MLPF-WB-04D3:BGA6C50P3X2_160X100X68, symbol MLPF-WB-04D3:MLPF-WB-04D3
- removed R1: 10k, Resistor_SMD:R_0402_1005Metric, symbol Device:R
- removed U1: STM32WBA52KGUx, Package_DFN_QFN:QFN-32-1EP_5x5mm_P0.5mm_EP3.1x3.1mm_ThermalVias, symbol MCU_ST_STM32WB:STM32WBA52KGUx
- added C18: 20p, Capacitor_SMD:C_0402_1005Metric, symbol Device:C
- added C19, C27, C29, C7: 100n, Capacitor_SMD:C_0402_1005Metric, symbol Device:C
- added C20, C21: 4.7u, Capacitor_SMD:C_0402_1005Metric, symbol Device:C
- added C28: 1u, Capacitor_SMD:C_0402_1005Metric, symbol Device:C
- added C30: 3p, Capacitor_SMD:C_0201_0603Metric, symbol Device:C
- added C31: 220n, Capacitor_SMD:C_0402_1005Metric, symbol Device:C
- added IC3: MLPF-NRG-01D3, MLPF-NRG-01D3:MLPFNRG01D3, symbol MLPF-NRG-01D3:MLPF-NRG-01D3
- added L1: LQG15HN22NG02D - 22n, Inductor_SMD:L_0402_1005Metric, symbol Device:L
- added L2: LQM21DN100M70L - 10u, Inductor_SMD:L_0805_2012Metric, symbol Device:L
- added L3: DNP, Inductor_SMD:L_0402_1005Metric, symbol Device:L
- added U4: STM32WB09KEVx, Package_DFN_QFN:QFN-32-1EP_5x5mm_P0.5mm_EP3.7x3.7mm, symbol MCU_ST_STM32WB:STM32WB09KEVx
- C1: value 1u -> DNP
- C15: value 100n -> 3p; footprint Capacitor_SMD:C_0402_1005Metric -> Capacitor_SMD:C_0201_0603Metric
- C2: value 10u -> DNP; footprint Capacitor_SMD:C_0603_1608Metric -> Capacitor_SMD:C_0402_1005Metric
- L4: value 2u2 -> 81-DFE201612E-2R2MP2 - 2u2
- Y1: value 32.768kHz -> 520-.327-6-1210-TR (32.768kHz)
- Y2: value 32MHz -> NX1612SA-32.000MHZ-CHP-CIS-3
Connections:
- net +1V8: now also C15.1, C19.1, C20.1, C21.1, C27.1, C28.1, C29.1, C30.1, C7.1, L2.1, U4.13 (VDD), U4.15 (VDDRF), U4.24 (VDDSD), U4.27 (VFBSD), U4.32 (VDD); no longer C2.1
- net BATT_ADC: now also U4.3 (PB1)
- net BATT_EN: now also U4.2 (PB2)
- net CRYSTAL1: now also U4.21 (PB12)
- net CRYSTAL2: now also U4.20 (PB13)
- net GND: now also R3.2, C19.2, C20.2, C21.2, C27.2, C28.2, C29.2, C30.2, C31.2, C7.2, IC3.A2 (GND4), IC3.B1 (GND3), IC3.B2 (GND2), IC3.B3 (GND1), U4.26 (VSSSD); no longer R3.1
- net IMU_INT: now also U4.8 (PA0)
- net MISO: now also U4.9 (PA8)
- net MOSI: now also U4.12 (PA11)
- net OSC_IN: now also U4.17 (OSCIN)
- net OSC_OUT: now also U4.16 (OSCOUT)
- net RF: now also C18.1, IC3.A3 (IN)
- net SCLK: now also U4.1 (PB3)
- net SWCLK: now also U4.5 (PA3)
- net SWDIO: now also U4.6 (PA2)
- net ~{RESET}: now also U4.29 (RSTN)
- net ~{SS}: now also U4.10 (PA9)
- net at C1.1: now also C2.1, IC3.A1 (OUT), L3.1
- net at E1.1: now also L3.2
- net SWO renamed UART_TX
- net UART_TX: now also U4.7 (PA1)
- new net: L1.1, L2.2
- new net: R3.1, U4.11 (PA10)
- new net: C18.2, U4.14 (RF1)
- new net VDD_CAP: C31.1, U4.28 (VDDA_VCAP)
- new net VLXSD: L1.2, U4.25 (VLXSD)
- no-connect marks 2 -> 3
Other:
- note added: "Internal load caps"
- note added: "Is this needed?"
- note added: "LQM18DN100M70L"
- note added: "UART_RX"
- note added: "VDD (13)"
- note added: "VDD (32)"
- note added: "VDDRF (15)"
- note added: "VDDSD (24)"
- note removed: "520-.327-6-1210-TR"
- note removed: "609-2450AT42E0100001"
- note removed: "81-DFE201612E-2R2MP2"
- note removed: "Caps needed?"
- note removed: "Debugging"
- note removed: "MCU"
- note removed: "MLPF-WB-04D3"
- note removed: "NX1612SA-32.000MHZ-CHP-CIS-3"
- note removed: "SPI"
- note removed: "To calculate"
- note removed: "needed?"
- moved on the sheet: C12, C13, C26, D1, J1, R2, R4, R5, Y1, Y2

Commit message: Hardware design, almost finished
Connections:
- net +BATT: no longer B1.2
- net BATT_EN: now also U4.4 (PB0); no longer U4.2 (PB2)
- net IMU_INT: now also U4.2 (PB2); no longer U4.8 (PA0)
- no-connect marks 3 -> 4
Changed lines of the file:
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@@
 	)
 	(no_connect
+		(at 26.67 25.4)
+	)
+	(no_connect
 		(at 185.42 146.05)
 	)
@@
 	(wire
 		(pts
+			(xy 185.42 120.65) (xy 204.47 120.65)
+		)
+		(stroke
+			(width 0)
+			(type default)
+		)
+	)
+	(wire
+		(pts
 			(xy 130.81 113.03) (xy 149.86 113.03)
 		)
@@
 	(wire
 		(pts
-			(xy 185.42 125.73) (xy 204.47 125.73)
-		)
-		(stroke
-			(width 0)
-			(type default)
-		)
-	)
-	(wire
-		(pts
 			(xy 48.26 115.57) (xy 48.26 114.3)
 		)
@@
 	(wire
 		(pts
-			(xy 185.42 97.79) (xy 204.47 97.79)
-		)
-		(stroke
-			(width 0)
-			(type default)
-		)
-	)
-	(wire
-		(pts
 			(xy 252.73 25.4) (xy 252.73 27.94)
 		)
@@
 	(wire
 		(pts
+			(xy 185.42 125.73) (xy 204.47 125.73)
+		)
+		(stroke
+			(width 0)
+			(type default)
+		)
+	)
+	(wire
+		(pts
 			(xy 73.66 163.83) (xy 64.77 163.83)
 		)
@@
 	(label "UART_TX"
 		(at 245.11 38.1 0)
-		(fields_autoplaced yes)
 		(effects
 			(font
@@
 	(label "CRYSTAL1"
 		(at 208.28 140.97 180)
-		(fields_autoplaced yes)
 		(effects
 			(font
@@
 	(label "BATT_EN"
 		(at 22.86 189.23 0)
-		(fields_autoplaced yes)
 		(effects
 			(font
@@
 	(label "SW_IMU"
 		(at 46.99 72.39 0)
-		(fields_autoplaced yes)
 		(effects
 			(font
@@
 	(label "SW_BATT"
 		(at 92.71 165.1 180)
-		(fields_autoplaced yes)
 		(effects
 			(font
@@
 	(label "CRYSTAL2"
 		(at 160.02 20.32 270)
-		(fields_autoplaced yes)
 		(effects
 			(font
@@
 	(label "~{RESET}"
 		(at 130.81 97.79 0)
-		(fields_autoplaced yes)
 		(effects
 			(font
@@
 	(label "LED"
 		(at 162.56 182.88 180)
-		(fields_autoplaced yes)
 		(effects
 			(font
@@
 	(label "OSC_OUT"
 		(at 130.81 113.03 0)
-		(fields_autoplaced yes)
 		(effects
 			(font
@@
 	(label "IMU_INT"
 		(at 82.55 93.98 180)
-		(fields_autoplaced yes)
 		(effects
 			(font
@@
 	(label "SWCLK"
 		(at 204.47 105.41 180)
-		(fields_autoplaced yes)
 		(effects
 			(font
@@
 	(label "VDD_CAP"
 		(at 176.53 76.2 180)
-		(fields_autoplaced yes)
 		(effects
 			(font
@@
 	(label "~{RESET}"
 		(at 245.11 33.02 0)
-		(fields_autoplaced yes)
 		(effects
 			(font
@@
 	(label "RF"
 		(at 115.57 115.57 0)
-		(fields_autoplaced yes)
 		(effects
 			(font
@@
 		)
 	)
-	(label "BATT_EN"
-		(at 204.47 125.73 180)
-		(fields_autoplaced yes)
-		(effects
-			(font
-				(size 1.27 1.27)
-			)
-			(justify right bottom)
-		)
-	)
 	(label "SW_IMU"
 		(at 73.66 163.83 180)
-		(fields_autoplaced yes)
 		(effects
 			(font
@@
 	(label "SWDIO"
 		(at 204.47 102.87 180)
-		(fields_autoplaced yes)
 		(effects
 			(font
@@
 	(label "UART_TX"
 		(at 204.47 100.33 180)
-		(fields_autoplaced yes)
 		(effects
 			(font
@@
 	(label "BATT_ADC"
 		(at 80.01 179.07 0)
-		(fields_autoplaced yes)
 		(effects
 			(font
@@
 	(label "~{RESET}"
 		(at 231.14 40.64 0)
-		(fields_autoplaced yes)
 		(effects
 			(font
@@
 		)
 	)
+	(label "IMU_INT"
+		(at 204.47 125.73 180)
+		(effects
+			(font
+				(size 1.27 1.27)
+			)
+			(justify right bottom)
+		)
+	)
 	(label "SCLK"
 		(at 19.05 97.79 0)
-		(fields_autoplaced yes)
 		(effects
 			(font
@@
 	(label "LED"
 		(at 60.96 139.7 0)
-		(fields_autoplaced yes)
 		(effects
 			(font
@@
 	(label "SWDIO"
 		(at 245.11 30.48 0)
-		(fields_autoplaced yes)
 		(effects
 			(font
@@
 	(label "SWCLK"
 		(at 245.11 35.56 0)
-		(fields_autoplaced yes)
 		(effects
 			(font
@@
 	(label "OSC_OUT"
 		(at 201.93 26.67 180)
-		(fields_autoplaced yes)
 		(effects
 			(font
@@
 	(label "VDD_CAP"
 		(at 212.09 83.82 0)
-		(fields_autoplaced yes)
 		(effects
 			(font
@@
 	(label "MISO"
 		(at 19.05 102.87 0)
-		(fields_autoplaced yes)
 		(effects
 			(font
@@
 	(label "BATT_ADC"
 		(at 204.47 123.19 180)
-		(fields_autoplaced yes)
 		(effects
 			(font
@@
 		)
 	)
-	(label "OSC_IN"
-		(at 166.37 26.67 0)
-		(fields_autoplaced yes)
+	(label "BATT_EN"
+		(at 204.47 120.65 180)
 		(effects
 			(font
 				(size 1.27 1.27)
 			)
-			(justify left bottom)
+			(justify right bottom)
 		)
 	)
-	(label "IMU_INT"
-		(at 204.47 97.79 180)
-		(fields_autoplaced yes)
+	(label "OSC_IN"
+		(at 166.37 26.67 0)
 		(effects
 			(font
 				(size 1.27 1.27)
 			)
-			(justify right bottom)
+			(justify left bottom)
 		)
 	)
 	(label "IMU_EN"
 		(at 162.56 177.8 180)
-		(fields_autoplaced yes)
 		(effects
 			(font
@@
 	(label "~{SS}"
 		(at 19.05 95.25 0)
-		(fields_autoplaced yes)
 		(effects
 			(font
@@
 	(label "VFBSD"
 		(at 130.81 105.41 0)
-		(fields_autoplaced yes)
 		(effects
 			(font
@@
 	(label "IMU_EN"
 		(at 22.86 168.91 0)
-		(fields_autoplaced yes)
 		(effects
 			(font
@@
 	(label "MISO"
 		(at 204.47 107.95 180)
-		(fields_autoplaced yes)
 		(effects
 			(font
@@
 	(label "VLXSD"
 		(at 130.81 100.33 0)
-		(fields_autoplaced yes)
 		(effects
 			(font
@@
 	(label "~{SS}"
 		(at 204.47 110.49 180)
-		(fields_autoplaced yes)
 		(effects
 			(font
@@
 	(label "VFBSD"
 		(at 275.59 86.36 180)
-		(fields_autoplaced yes)
 		(effects
 			(font
@@
 	(label "CRYSTAL2"
 		(at 208.28 143.51 180)
-		(fields_autoplaced yes)
 		(effects
 			(font
@@
 	(label "OSC_IN"
 		(at 130.81 110.49 0)
-		(fields_autoplaced yes)
 		(effects
 			(font
@@
 	(label "SCLK"
 		(at 204.47 128.27 180)
-		(fields_autoplaced yes)
 		(effects
 			(font
@@
 	(label "SW_BATT"
 		(at 73.66 184.15 180)
-		(fields_autoplaced yes)
 		(effects
 			(font
@@
 	(label "CRYSTAL1"
 		(at 144.78 20.32 270)
-		(fields_autoplaced yes)
 		(effects
 			(font
@@
 	(label "VLXSD"
 		(at 275.59 80.01 180)
-		(fields_autoplaced yes)
 		(effects
 			(font
@@
 	(label "MOSI"
 		(at 19.05 100.33 0)
-		(fields_autoplaced yes)
 		(effects
 			(font
@@
 	(label "MOSI"
 		(at 204.47 115.57 180)
-		(fields_autoplaced yes)
 		(effects
 			(font
@@
 	(label "RF"
 		(at 204.47 133.35 0)
-		(fields_autoplaced yes)
 		(effects
 			(font
@@
 		)
 		(property "Footprint" "Battery_holder:WA-BCMC_79523211"
-			(at 39.37 22.86 0)
+			(at 39.37 19.812 0)
 			(effects
 				(font
@@
 		)
 		(property "MF" "Würth Elektronik"
-			(at 39.37 22.86 0)
+			(at 39.37 14.478 0)
 			(effects
 				(font
@@
 		)
 		(property "SnapEDA_Link" "https://www.snapeda.com/parts/79523141/W%25C3%25BCrth+Elektronik+Midcom/view-part/?ref=snap"
-			(at 39.37 22.86 0)
+			(at 39.37 11.43 0)
 			(effects
 				(font
@@
 		)
 		(property "BATTERY-TYPE" "2016,2020,2025,2032"
-			(at 39.37 22.86 0)
+			(at 40.386 12.446 0)
 			(effects
 				(font
@@
 		)
 		(property "DATASHEET-URL" "https://www.we-online.com/redexpert/spec/79523141?ae"
-			(at 39.37 22.86 0)
+			(at 40.894 13.208 0)
 			(effects
 				(font
@@
 		)
 		(property "Check_prices" "https://www.snapeda.com/parts/79523141/W%25C3%25BCrth+Elektronik+Midcom/view-part/?ref=eda"
-			(at 39.37 22.86 0)
+			(at 39.37 9.398 0)
 			(effects
 				(font
