File: V2/Hardware/plant_sensor_v2/plant_sensor_v2.kicad_sch (KiCad schematic)
At the start: 43 parts, among them IC1 ICM-20948, IC3 MLPF-NRG-01D3, J1 TC2030_SWD-MCP-NL, U2 TPS22960RSER, U3 TPS62840DLCR, U4 STM32WB09KEVx, Y1 520-.327-6-1210-TR (32.768kHz), Y2 NX1612SA-32.000MHZ-CHP-CIS-3

Commit message: Update hardware
Connections:
- net IMU_EN: now also U4.23 (PB6)
- net LED: now also U4.8 (PA0)
Changed lines of the file:
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@@
+	(wire
+		(pts
+			(xy 185.42 97.79) (xy 204.47 97.79)
+		)
+		(stroke
+			(width 0)
+			(type default)
+		)
+	)
 	(wire
 		(pts
@@
 	(wire
 		(pts
-			(xy 162.56 177.8) (xy 148.59 177.8)
-		)
-		(stroke
-			(width 0)
-			(type default)
-		)
-	)
-	(wire
-		(pts
 			(xy 243.84 86.36) (xy 247.65 86.36)
 		)
@@
 	(wire
 		(pts
+			(xy 185.42 135.89) (xy 204.47 135.89)
+		)
+		(stroke
+			(width 0)
+			(type default)
+		)
+	)
+	(wire
+		(pts
 			(xy 219.71 113.03) (xy 217.17 113.03)
 		)
@@
 		(pts
 			(xy 92.71 165.1) (xy 92.71 171.45)
-		)
-		(stroke
-			(width 0)
-			(type default)
-		)
-	)
-	(wire
-		(pts
-			(xy 162.56 182.88) (xy 148.59 182.88)
 		)
 		(stroke
@@
 	(label "UART_TX"
 		(at 245.11 38.1 0)
+		(fields_autoplaced yes)
 		(effects
 			(font
@@
 	(label "CRYSTAL1"
 		(at 208.28 140.97 180)
+		(fields_autoplaced yes)
 		(effects
 			(font
@@
 	(label "BATT_EN"
 		(at 22.86 189.23 0)
+		(fields_autoplaced yes)
 		(effects
 			(font
@@
 	(label "SW_IMU"
 		(at 46.99 72.39 0)
+		(fields_autoplaced yes)
 		(effects
 			(font
@@
 	(label "SW_BATT"
 		(at 92.71 165.1 180)
+		(fields_autoplaced yes)
 		(effects
 			(font
@@
 	(label "CRYSTAL2"
 		(at 160.02 20.32 270)
+		(fields_autoplaced yes)
 		(effects
 			(font
@@
 	(label "~{RESET}"
 		(at 130.81 97.79 0)
+		(fields_autoplaced yes)
 		(effects
 			(font
@@
 	)
 	(label "LED"
-		(at 162.56 182.88 180)
+		(at 204.47 97.79 180)
+		(fields_autoplaced yes)
 		(effects
 			(font
@@
 	(label "OSC_OUT"
 		(at 130.81 113.03 0)
+		(fields_autoplaced yes)
 		(effects
 			(font
@@
 	(label "IMU_INT"
 		(at 82.55 93.98 180)
+		(fields_autoplaced yes)
 		(effects
 			(font
@@
 	(label "SWCLK"
 		(at 204.47 105.41 180)
+		(fields_autoplaced yes)
 		(effects
 			(font
@@
 	(label "VDD_CAP"
 		(at 176.53 76.2 180)
+		(fields_autoplaced yes)
 		(effects
 			(font
@@
 	(label "~{RESET}"
 		(at 245.11 33.02 0)
+		(fields_autoplaced yes)
 		(effects
 			(font
@@
 	(label "RF"
 		(at 115.57 115.57 0)
+		(fields_autoplaced yes)
 		(effects
 			(font
@@
 	(label "SW_IMU"
 		(at 73.66 163.83 180)
+		(fields_autoplaced yes)
+		(effects
+			(font
+				(size 1.27 1.27)
+			)
+			(justify right bottom)
+		)
+	)
+	(label "IMU_EN"
+		(at 204.47 135.89 180)
+		(fields_autoplaced yes)
 		(effects
 			(font
@@
 	(label "SWDIO"
 		(at 204.47 102.87 180)
+		(fields_autoplaced yes)
 		(effects
 			(font
@@
 	(label "UART_TX"
 		(at 204.47 100.33 180)
+		(fields_autoplaced yes)
 		(effects
 			(font
@@
 	(label "BATT_ADC"
 		(at 80.01 179.07 0)
+		(fields_autoplaced yes)
 		(effects
 			(font
@@
 	(label "~{RESET}"
 		(at 231.14 40.64 0)
+		(fields_autoplaced yes)
 		(effects
 			(font
@@
 	(label "IMU_INT"
 		(at 204.47 125.73 180)
+		(fields_autoplaced yes)
 		(effects
 			(font
@@
 	(label "SCLK"
 		(at 19.05 97.79 0)
+		(fields_autoplaced yes)
 		(effects
 			(font
@@
 	(label "LED"
 		(at 60.96 139.7 0)
+		(fields_autoplaced yes)
 		(effects
 			(font
@@
 	(label "SWDIO"
 		(at 245.11 30.48 0)
+		(fields_autoplaced yes)
 		(effects
 			(font
@@
 	(label "SWCLK"
 		(at 245.11 35.56 0)
+		(fields_autoplaced yes)
 		(effects
 			(font
@@
 	(label "OSC_OUT"
 		(at 201.93 26.67 180)
+		(fields_autoplaced yes)
 		(effects
 			(font
@@
 	(label "VDD_CAP"
 		(at 212.09 83.82 0)
+		(fields_autoplaced yes)
 		(effects
 			(font
@@
 	(label "MISO"
 		(at 19.05 102.87 0)
+		(fields_autoplaced yes)
 		(effects
 			(font
@@
 	(label "BATT_ADC"
 		(at 204.47 123.19 180)
+		(fields_autoplaced yes)
 		(effects
 			(font
@@
 	(label "BATT_EN"
 		(at 204.47 120.65 180)
+		(fields_autoplaced yes)
 		(effects
 			(font
@@
 	(label "OSC_IN"
 		(at 166.37 26.67 0)
+		(fields_autoplaced yes)
 		(effects
 			(font
@@
 			)
 			(justify left bottom)
-		)
-	)
-	(label "IMU_EN"
-		(at 162.56 177.8 180)
-		(effects
-			(font
-				(size 1.27 1.27)
-			)
-			(justify right bottom)
 		)
 	)
 	(label "~{SS}"
 		(at 19.05 95.25 0)
+		(fields_autoplaced yes)
 		(effects
 			(font
@@
 	(label "VFBSD"
 		(at 130.81 105.41 0)
+		(fields_autoplaced yes)
 		(effects
 			(font
@@
 	(label "IMU_EN"
 		(at 22.86 168.91 0)
+		(fields_autoplaced yes)
 		(effects
 			(font
@@
 	(label "MISO"
 		(at 204.47 107.95 180)
+		(fields_autoplaced yes)
 		(effects
 			(font
@@
 	(label "VLXSD"
 		(at 130.81 100.33 0)
+		(fields_autoplaced yes)
 		(effects
 			(font
@@
 	(label "~{SS}"
 		(at 204.47 110.49 180)
+		(fields_autoplaced yes)
 		(effects
 			(font
@@
 	(label "VFBSD"
 		(at 275.59 86.36 180)
+		(fields_autoplaced yes)
 		(effects
 			(font
@@
 	(label "CRYSTAL2"
 		(at 208.28 143.51 180)
+		(fields_autoplaced yes)
 		(effects
 			(font
@@
 	(label "OSC_IN"
 		(at 130.81 110.49 0)
+		(fields_autoplaced yes)
 		(effects
 			(font
@@
 	(label "SCLK"
 		(at 204.47 128.27 180)
+		(fields_autoplaced yes)
 		(effects
 			(font
@@
 	(label "SW_BATT"
 		(at 73.66 184.15 180)
+		(fields_autoplaced yes)
 		(effects
 			(font
@@
 	(label "CRYSTAL1"
 		(at 144.78 20.32 270)
+		(fields_autoplaced yes)
 		(effects
 			(font
@@
 	(label "VLXSD"
 		(at 275.59 80.01 180)
+		(fields_autoplaced yes)
 		(effects
 			(font
@@
 	(label "MOSI"
 		(at 19.05 100.33 0)
+		(fields_autoplaced yes)
 		(effects
 			(font
@@
 	(label "MOSI"
 		(at 204.47 115.57 180)
+		(fields_autoplaced yes)
 		(effects
 			(font
@@
 	(label "RF"
 		(at 204.47 133.35 0)
+		(fields_autoplaced yes)
 		(effects
 			(font
@@
 			)
 		)
-		(property "Datasheet" ""
+		(property "Datasheet" "https://www.mouser.be/datasheet/2/611/2450AT42E0100-1519638.pdf"
 			(at 269.24 133.35 0)
 			(effects
