File: V2/Hardware/plant_sensor_v2/plant_sensor_v2.kicad_sch (KiCad schematic)
At the start: 43 parts, among them IC1 ICM-20948, IC3 MLPF-NRG-01D3, J1 TC2030_SWD-MCP-NL, U2 TPS22960RSER, U3 TPS62840DLCR, U4 STM32WB09KEVx, Y1 520-.327-6-1210-TR (32.768kHz), Y2 NX1612SA-32.000MHZ-CHP-CIS-3

Commit message: Hardware V2 Finished
Parts:
- added TP1, TP10, TP11, TP2, TP4, TP5, TP6, TP7, TP8, TP9: TestPoint, TestPoint:TestPoint_Pad_D1.0mm, symbol Connector:TestPoint
Connections:
- net +1V8: now also TP1.1; no longer C26.1
- net GND: now also C26.1, U4.33 (VSS_EXPOSED), TP10.1, TP11.1
- net IMU_INT: now also TP4.1
- net MISO: now also TP8.1
- net MOSI: now also TP7.1
- net SCLK: now also TP6.1
- net SW_IMU: now also TP2.1
- net UART_TX: now also TP9.1
- net ~{SS}: now also TP5.1
- no-connect marks 4 -> 8
Other:
- moved on the sheet: C26

Commit message: BOM
Parts:
- U4: value STM32WB09KEVx -> STM32WB09KEV6TR
Other:
- note added: "79523211"
- note added: "81-GRM155R60G106ME5D"
Changed lines of the file:
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@@
+		)
+	)
+	(text "79523211"
+		(exclude_from_sim no)
+		(at 50.8 17.78 0)
+		(effects
+			(font
+				(size 1.27 1.27)
+			)
 		)
 	)
@@
 		(exclude_from_sim no)
 		(at 179.324 52.07 0)
+		(effects
+			(font
+				(size 1.27 1.27)
+			)
+		)
+	)
+	(text "81-GRM155R60G106ME5D"
+		(exclude_from_sim no)
+		(at 118.364 37.846 90)
 		(effects
 			(font
@@
 			)
 		)
-		(property "Value" "STM32WB09KEVx"
+		(property "Value" "STM32WB09KEV6TR"
 			(at 169.8341 158.75 0)
 			(effects

Commit message: Hardware update
Other:
- note added: "TODO: Add TPL5010 as RTC + WDT"
Changed lines of the file:
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@@
+		)
+	)
+	(text "TODO:\nAdd TPL5010 as RTC + WDT\n"
+		(exclude_from_sim no)
+		(at 139.446 175.768 0)
+		(effects
+			(font
+				(size 1.27 1.27)
+			)
+			(justify left)
 		)
 	)
