File: V2/Hardware/plant_sensor_v2/plant_sensor_v2.kicad_pcb (KiCad board)
At the start: 2 copper layers, 1 part, among them U1 STM32WBA52KGUx

Commit message: update hardware
Parts:
- added B1: WA-BCMC, Battery_holder:WA-BCMC_79523211, F.Cu at (192.2, 125.3)
- added C1: 1u, Capacitor_SMD:C_0402_1005Metric, F.Cu at (139.5, 101.3)
- added C10: 100n, Capacitor_SMD:C_0402_1005Metric, F.Cu at (161.6, 100.9)
- added C11: 100n, Capacitor_SMD:C_0402_1005Metric, F.Cu at (157.5, 103.3)
- added C12: 6p, Capacitor_SMD:C_0402_1005Metric, F.Cu at (143.6, 95.1)
- added C13: 6p, Capacitor_SMD:C_0402_1005Metric, F.Cu at (143.6, 98.8)
- added C14: 470n, Capacitor_SMD:C_0603_1608Metric, F.Cu at (133.4, 93.8)
- added C15: 100n, Capacitor_SMD:C_0402_1005Metric, F.Cu at (133.9, 95.1)
- added C16: 100n, Capacitor_SMD:C_0402_1005Metric, F.Cu at (133.9, 97.1)
- added C17: 4.7µ, Capacitor_SMD:C_0603_1608Metric, F.Cu at (133.6, 99.4)
- added C18: 1.5p, Capacitor_SMD:C_0402_1005Metric, F.Cu at (135.5, 91.8)
- added C19: 3.9p, Capacitor_SMD:C_0402_1005Metric, F.Cu at (135.5, 88.4)
- added C2: 10u, Capacitor_SMD:C_0603_1608Metric, F.Cu at (135.7, 102.4)
- added C20: 2.7p, Capacitor_SMD:C_0402_1005Metric, F.Cu at (135.5, 85.0)
- added C21: 6p, Capacitor_SMD:C_0402_1005Metric, F.Cu at (130.9, 94.2)
- added C22: 4.7u, Capacitor_SMD:C_0402_1005Metric, F.Cu at (137.2, 112.9)
- added C23: 10u, Capacitor_SMD:C_0402_1005Metric, F.Cu at (139.7, 111.6)
- added C24: 100n, Capacitor_SMD:C_0402_1005Metric, F.Cu at (152.2, 99.7)
- added C25: 100n, Capacitor_SMD:C_0402_1005Metric, F.Cu at (152.2, 101.7)
- added C26: 100n, Capacitor_SMD:C_0402_1005Metric, F.Cu at (167.6, 92.6)
- added C3: 100n, Capacitor_SMD:C_0402_1005Metric, F.Cu at (133.9, 98.2)
- added C4: 100n, Capacitor_SMD:C_0402_1005Metric, F.Cu at (137.1, 91.4)
- added C5: 100n, Capacitor_SMD:C_0402_1005Metric, F.Cu at (143.5, 94.1)
- added C6: 100n, Capacitor_SMD:C_0402_1005Metric, F.Cu at (139.5, 100.3)
- added C7: 6p, Capacitor_SMD:C_0402_1005Metric, F.Cu at (130.9, 98.2)
- added C8: 10n, Capacitor_SMD:C_0402_1005Metric, F.Cu at (174.3, 71.0)
- added C9: 100n, Capacitor_SMD:C_0402_1005Metric, F.Cu at (158.5, 103.3)
- added D1: LED, RED, LED_SMD:LED_0603_1608Metric, F.Cu at (120.3, 102.2)
- added FB1: 47R @ 100Mhz, Resistor_SMD:R_0402_1005Metric, F.Cu at (139.0, 102.7)
- added IC1: ICM-20948, Libraries:ICM20948, F.Cu at (158.0, 99.8)
- added J1: TC2030_SWD-MCP-NL, Connector:Tag-Connect_TC2030-IDC-NL_2x03_P1.27mm_Vertical, F.Cu at (167.4, 88.9)
- added L1: 1.3n, Inductor_SMD:L_0402_1005Metric, F.Cu at (135.0, 86.7)
- added L2: 1.8n, Inductor_SMD:L_0402_1005Metric, F.Cu at (135.0, 90.1)
- added L4: 2u2, Inductor_SMD:L_Murata_DFE201610P, F.Cu at (142.2, 112.9)
- added R1: 10k, Resistor_SMD:R_0402_1005Metric, F.Cu at (167.6, 91.6)
- added R2: R, Resistor_SMD:R_0402_1005Metric, F.Cu at (123.2, 102.2)
- added R3: 100k, Resistor_SMD:R_0402_1005Metric, F.Cu at (138.1, 91.4)
- added R4: 470k, Resistor_SMD:R_0402_1005Metric, F.Cu at (174.2, 69.0)
- added R5: 220k, Resistor_SMD:R_0402_1005Metric, F.Cu at (174.2, 70.0)
- added R6: 0, Resistor_SMD:R_0402_1005Metric, F.Cu at (139.6, 115.9)
- added U2: TPS22960RSER, TPS22960:RSE0008A, F.Cu at (149.4, 100.8)
- added U3: TPS62840DLCR, TPS62840:VSON8_2P1X1P6_TEX, F.Cu at (139.5, 113.9)
- added Y1: 32.768kHz, Crystal:Crystal_SMD_2012-2Pin_2.0x1.2mm, F.Cu at (143.6, 96.9)
- added Y2: 32MHz, Crystal:Crystal_SMD_2016-4Pin_2.0x1.6mm, F.Cu at (131.1, 96.2)
- moved U1 1.71 mm to (138.5, 96.0), turned to 90 degrees
Connections:
- U1 pad 10: unconnected-(U1-PB9-Pad10) -> /MISO
- U1 pad 11: unconnected-(U1-PB8-Pad11) -> /MOSI
- U1 pad 12: unconnected-(U1-PC15-Pad12) -> /CRYSTAL2
- U1 pad 13: unconnected-(U1-PC14-Pad13) -> /CRYSTAL1
- U1 pad 14: unconnected-(U1-VDD-Pad14) -> +1V8
- U1 pad 16: unconnected-(U1-PB3-Pad16) -> /SWO
- U1 pad 18: unconnected-(U1-PA14-Pad18) -> /SWCLK
- U1 pad 19: unconnected-(U1-PA13-Pad19) -> /SWDIO
- U1 pad 2: unconnected-(U1-PA8-Pad2) -> /BATT_ADC
- U1 pad 21: unconnected-(U1-PB15-Pad21) -> /LED
- U1 pad 22: unconnected-(U1-PH3-Pad22) -> Net-(U1-PH3)
- U1 pad 23: unconnected-(U1-VDD-Pad23) -> +1V8
- U1 pad 24: unconnected-(U1-NRST-Pad24) -> /~{RESET}
- U1 pad 25: unconnected-(U1-RF-Pad25) -> /RF
- U1 pad 26: unconnected-(U1-VDDHPA-Pad26) -> Net-(U1-VDDHPA)
- U1 pad 27: unconnected-(U1-VDDRF-Pad27) -> Net-(U1-VDDRF)
- U1 pad 28: unconnected-(U1-OSC_OUT-Pad28) -> /OSC_OUT
- U1 pad 29: unconnected-(U1-OSC_IN-Pad29) -> /OSC_IN
- U1 pad 3: unconnected-(U1-PA7-Pad3) -> /BATT_EN
- U1 pad 30: unconnected-(U1-VDDRFPA-Pad30) -> Net-(U1-VDDRFPA)
- U1 pad 31: unconnected-(U1-VDD-Pad31) -> +1V8
- U1 pad 32: unconnected-(U1-VCAP-Pad32) -> Net-(U1-VCAP)
- U1 pad 4: unconnected-(U1-PA6-Pad4) -> /IMU_EN
- U1 pad 5: unconnected-(U1-VDDA-Pad5) -> Net-(U1-VDDA)
- U1 pad 6: unconnected-(U1-PA5-Pad6) -> /~{SS}
- U1 pad 8: unconnected-(U1-PA1-Pad8) -> /IMU_INT
- U1 pad 9: unconnected-(U1-PA0-Pad9) -> /SCLK
Routing:
- net +BATT: track 0.00 -> 5.85 mm
- net GND: track 0.00 -> 5.15 mm, vias 0 -> 6
- net Net-(U3-SW): track 0.00 -> 2.03 mm
- net +1V8: track 0.00 -> 1.64 mm
- net Net-(U3-VSET): track 0.00 -> 1.25 mm
- added copper zone on F.Cu, net +1V8
- added copper zone on F.Cu, net +BATT

Commit message: update hardware
Parts:
- B1: moved to B.Cu
- moved B1 104.1 mm to (102.9, 72.0), turned to 180 degrees
- moved C26 78.0 mm to (93.0, 69.8)
- moved R1 78.0 mm to (93.0, 68.8)
- moved J1 76.4 mm to (94.4, 66.3), turned to 180 degrees
- moved R5 63.2 mm to (111.1, 67.6)
- moved C8 63.2 mm to (111.1, 68.6)
- moved R4 63.2 mm to (111.0, 66.7)
- moved C10 54.3 mm to (112.0, 78.8)
- moved C11 54.3 mm to (107.9, 81.1)
- moved IC1 54.3 mm to (108.4, 77.7)
- moved C9 54.3 mm to (108.9, 81.2)
- moved L4 53.0 mm to (100.7, 80.0)
- moved R6 53.0 mm to (98.1, 82.9)
- moved U3 53.0 mm to (98.0, 80.9)
- moved C22 53.0 mm to (95.7, 79.9)
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Other:
- board outline added: 28.6 x 28.6 mm

Commit message: update hardware
Parts:
- removed C18: 1.5p, Capacitor_SMD:C_0402_1005Metric
- removed C19: 3.9p, Capacitor_SMD:C_0402_1005Metric
- removed C20: 2.7p, Capacitor_SMD:C_0402_1005Metric
- removed L1: 1.3n, Inductor_SMD:L_0402_1005Metric
- removed L2: 1.8n, Inductor_SMD:L_0402_1005Metric
- added E1: 609-2450AT42E0100001, Antenna:XDCR_2450AT42E0100E, F.Cu at (102.9, 61.5)
- added IC2: MLPF-WB-04D3, MLPF-WB-04D3:BGA6C50P3X2_160X100X68, F.Cu at (98.3, 64.0)
- moved C26 59.3 mm to (105.7, 127.8)
- moved R1 59.3 mm to (105.7, 126.7)
- moved C8 53.5 mm to (106.0, 121.9)
- moved R4 53.5 mm to (105.9, 120.0)
- moved R5 53.5 mm to (105.9, 120.9)
- moved D1 52.3 mm to (104.9, 116.8)
- moved R2 52.3 mm to (107.8, 116.8)
- moved C2 43.2 mm to (97.8, 119.6)
- moved J1 15.5 mm to (109.8, 65.0), turned to -45 degrees
- moved C7 4.06 mm to (98.8, 72.3), turned to 90 degrees
- moved FB1 2.80 mm to (103.9, 76.0), turned to 0 degrees
- moved C17 2.76 mm to (100.6, 74.7), turned to -90 degrees
- moved C5 2.53 mm to (107.7, 67.6)
- moved C12 2.53 mm to (107.8, 68.6)
- moved C13 2.53 mm to (107.8, 72.3)
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Routing:
- net /SWO: track 0.00 -> 10.4 mm, vias 0 -> 2
- net /SWCLK: track 0.00 -> 9.90 mm, vias 0 -> 2
- net /SWDIO: track 0.00 -> 9.87 mm, vias 0 -> 2
- net /RF: track 0.00 -> 5.17 mm
- net +1V8: track 1.64 -> 6.43 mm
- net GND: track 5.15 -> 9.83 mm, vias 6 -> 36
- net /CRYSTAL2: track 0.00 -> 4.20 mm
- net Net-(IC2-OUT): track 0.00 -> 4.13 mm
- net +BATT: track 5.85 -> 1.73 mm
- net /CRYSTAL1: track 0.00 -> 3.82 mm
- net Net-(U1-VDDA): track 0.00 -> 3.80 mm
- net Net-(U1-VCAP): track 0.00 -> 2.46 mm
- net Net-(U1-PH3): track 0.00 -> 1.83 mm
- net /OSC_OUT: track 0.00 -> 1.56 mm
- net /OSC_IN: track 0.00 -> 1.32 mm
- added copper zone on B.Cu, net GND
- added copper zone on F.Cu, net GND
- added copper zone on In1.Cu, net GND
- added copper zone on In2.Cu, net GND
Other:
- board size 28.6 x 28.6 mm -> 24.7 x 24.7 mm
- copper layers 2 -> 4

Commit message: update hardware
Parts:
- removed C21, C7: 6p, Capacitor_SMD:C_0402_1005Metric
- Y1: footprint Crystal:Crystal_SMD_2012-2Pin_2.0x1.2mm -> Crystal3:XTAL_ECS-.327-6-1210-TR
- Y2: footprint Crystal:Crystal_SMD_2016-4Pin_2.0x1.6mm -> Crystal2:OSCSC105P160X120X35-4N
- moved Y2 1.24 mm to (98.2, 71.9)
- moved C13 0.64 mm to (107.8, 71.6)
- moved Y1 0.34 mm to (107.8, 70.1)
Routing:
- net /CRYSTAL2: track 4.20 -> 0.00 mm
- net /CRYSTAL1: track 3.82 -> 0.00 mm
- net /OSC_OUT: track 1.56 -> 0.00 mm
- net /OSC_IN: track 1.32 -> 0.00 mm

Commit message: hardware update
Parts:
- removed C14: 470n, Capacitor_SMD:C_0603_1608Metric
- removed C16, C3, C4, C5, C6: 100n, Capacitor_SMD:C_0402_1005Metric
- removed C17: 4.7µ, Capacitor_SMD:C_0603_1608Metric
- removed C8: 10n, Capacitor_SMD:C_0402_1005Metric
- removed FB1: 47R @ 100Mhz, Resistor_SMD:R_0402_1005Metric
- removed IC2: MLPF-WB-04D3, MLPF-WB-04D3:BGA6C50P3X2_160X100X68
- removed R1: 10k, Resistor_SMD:R_0402_1005Metric
- removed U1: STM32WBA52KGUx, Package_DFN_QFN:QFN-32-1EP_5x5mm_P0.5mm_EP3.1x3.1mm_ThermalVias
- added C18: 20p, Capacitor_SMD:C_0402_1005Metric, F.Cu at (99.7, 69.0)
- added C19: 100n, Capacitor_SMD:C_0402_1005Metric, F.Cu at (99.0, 77.1)
- added C20: 4.7u, Capacitor_SMD:C_0402_1005Metric, F.Cu at (99.0, 78.1)
- added C21: 4.7u, Capacitor_SMD:C_0402_1005Metric, F.Cu at (95.7, 75.6)
- added C27: 100n, Capacitor_SMD:C_0402_1005Metric, F.Cu at (96.7, 75.6)
- added C28: 1u, Capacitor_SMD:C_0402_1005Metric, F.Cu at (103.8, 77.1)
- added C29: 100n, Capacitor_SMD:C_0402_1005Metric, F.Cu at (102.4, 66.8)
- added C30: 3p, Capacitor_SMD:C_0201_0603Metric, F.Cu at (102.3, 67.8)
- added C31: 220n, Capacitor_SMD:C_0402_1005Metric, F.Cu at (100.6, 77.7)
- added C7: 100n, Capacitor_SMD:C_0402_1005Metric, F.Cu at (97.0, 68.6)
- added IC3: MLPF-NRG-01D3, MLPF-NRG-01D3:MLPFNRG01D3, F.Cu at (99.8, 66.2)
- added L1: LQG15HN22NG02D - 22n, Inductor_SMD:L_0402_1005Metric, F.Cu at (97.3, 77.6)
- added L2: LQM21DN100M70L - 10u, Inductor_SMD:L_0805_2012Metric, F.Cu at (98.3, 79.7)
- added L3: DNP, Inductor_SMD:L_0402_1005Metric, F.Cu at (99.6, 63.5)
- added U4: STM32WB09KEVx, Package_DFN_QFN:QFN-32-1EP_5x5mm_P0.5mm_EP3.7x3.7mm, F.Cu at (100.6, 73.3)
- C1: value 1u -> DNP
- C15: value 100n -> 3p; footprint Capacitor_SMD:C_0402_1005Metric -> Capacitor_SMD:C_0201_0603Metric
- C2: value 10u -> DNP; footprint Capacitor_SMD:C_0603_1608Metric -> Capacitor_SMD:C_0402_1005Metric
- L4: value 2u2 -> 81-DFE201612E-2R2MP2 - 2u2
- Y1: value 32.768kHz -> 520-.327-6-1210-TR (32.768kHz)
- Y2: value 32MHz -> NX1612SA-32.000MHZ-CHP-CIS-3
- moved C2 56.6 mm to (98.0, 63.0)
- moved R2 51.6 mm to (104.9, 65.3), turned to 90 degrees
- moved D1 51.6 mm to (102.8, 65.3)
- moved C26 50.2 mm to (101.6, 77.7), turned to 90 degrees
- moved R4 42.9 mm to (106.7, 77.0)
- moved R5 42.9 mm to (106.7, 78.0)
- moved C12 14.5 mm to (94.5, 74.3), turned to -90 degrees
- moved C13 13.3 mm to (94.5, 72.5), turned to 90 degrees
- moved C1 12.3 mm to (98.0, 64.0), turned to 180 degrees
- moved Y1 12.2 mm to (96.0, 73.3), turned to 90 degrees
- moved C22 11.2 mm to (106.2, 81.3), turned to -90 degrees
- moved C24 8.59 mm to (110.8, 78.2)
- moved C23 8.20 mm to (103.7, 82.6), turned to 0 degrees
- moved R6 6.49 mm to (103.8, 78.3), turned to 0 degrees
- moved U2 6.17 mm to (109.0, 77.5), turned to 180 degrees
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Connections:
- C1 pad 1: Net-(U1-VDDA) -> Net-(IC3-OUT)
- C15 pad 1: Net-(U1-VDDRF) -> +1V8
- C2 pad 1: +1V8 -> Net-(IC3-OUT)
- J1 pad 6: /SWO -> /UART_TX
- R3 pad 1: GND -> Net-(U4-PA10)
- R3 pad 2: Net-(U1-PH3) -> GND
Routing:
- net +1V8: track 6.43 -> 42.5 mm, vias 0 -> 2
- net +BATT: track 1.73 -> 20.9 mm
- net /UART_TX: track 0.00 -> 17.2 mm, vias 0 -> 2
- net /MISO: track 0.00 -> 12.6 mm, vias 0 -> 2
- net /MOSI: track 0.00 -> 12.0 mm, vias 0 -> 2
- net GND: track 9.83 -> 20.6 mm
- net /~{SS}: track 0.00 -> 10.7 mm, vias 0 -> 2
- net /SCLK: track 0.00 -> 10.6 mm, vias 0 -> 2
- net /SWO: track 10.4 -> 0.00 mm, vias 2 -> 0
- net /SW_IMU: track 0.00 -> 9.80 mm
- net /BATT_EN: track 0.00 -> 9.09 mm, vias 0 -> 2
- net /BATT_ADC: track 0.00 -> 8.08 mm, vias 0 -> 2
- net Net-(U4-PA10): track 0.00 -> 5.23 mm
- net /SWCLK: track 9.90 -> 14.3 mm
- net /SWDIO: track 9.87 -> 14.2 mm
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
Commit message: Hardware design, almost finished
Parts:
- moved R3 0.70 mm to (105.0, 67.2), turned to 90 degrees
Connections:
- B1 pad 2: +BATT -> unconnected-(B1-Pad2)
- U4 pad 2: /BATT_EN -> /IMU_INT
- U4 pad 4: unconnected-(U4-PB0-Pad4) -> /BATT_EN
- U4 pad 8: /IMU_INT -> unconnected-(U4-PA0-Pad8)
Routing:
- net +1V8: track 42.5 -> 87.9 mm, vias 2 -> 8
- net /~{RESET}: track 1.76 -> 19.2 mm, vias 0 -> 2
- net GND: track 20.6 -> 35.0 mm, vias 36 -> 102
- net /IMU_INT: track 0.00 -> 8.99 mm, vias 0 -> 2
- net /SCLK: track 10.6 -> 8.39 mm
- net /BATT_EN: track 9.09 -> 11.1 mm
- net /MISO: track 12.6 -> 10.6 mm
- net /~{SS}: track 10.7 -> 8.97 mm
- net +BATT: track 20.9 -> 22.2 mm, vias 0 -> 1
- net /MOSI: track 12.0 -> 10.7 mm, vias 2 -> 0
- net Net-(U4-PA10): track 5.23 -> 5.38 mm, vias 0 -> 2
Other:
- board size 24.7 x 24.7 mm -> 25.3 x 25.3 mm

Commit message: Update hardware
Connections:
- U4 pad 23: unconnected-(U4-PB6-Pad23) -> /IMU_EN
- U4 pad 8: unconnected-(U4-PA0-Pad8) -> /LED
Routing:
- net /IMU_EN: track 0.00 -> 17.3 mm, vias 0 -> 2
- net /LED: track 0.00 -> 10.1 mm, vias 0 -> 2
- net +1V8: track 87.9 -> 89.1 mm
- net /MOSI: track 10.7 -> 10.1 mm
- net GND: vias 102 -> 100
- removed copper zone on F.Cu, net +1V8
Other:
- board text added: "Plantsensor LW Made by JC"
- board text added: "d"

Commit message: Hardware update
Routing:
- net GND: track 35.0 -> 37.1 mm, vias 100 -> 106
- net +1V8: track 89.1 -> 87.6 mm
- net /MOSI: track 10.1 -> 9.57 mm
Other:
- board size 25.3 x 25.3 mm -> 25.5 x 25.4 mm
