File: V2/Hardware/plant_sensor_v2/plant_sensor_v2.kicad_pcb (KiCad board)
At the start: 4 copper layers, 25.5 x 25.4 mm, 43 parts, among them IC1 ICM-20948, IC3 MLPF-NRG-01D3, J1 TC2030_SWD-MCP-NL, U2 TPS22960RSER, U3 TPS62840DLCR, U4 STM32WB09KEVx, Y1 520-.327-6-1210-TR (32.768kHz), Y2 NX1612SA-32.000MHZ-CHP-CIS-3

Commit message: update
Routing:
- net GND: vias 106 -> 118
Changed lines of the file:
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@@
 		(tags "TPS62840DLCR ")
 		(property "Reference" "U3"
-			(at -0.114 -1.736 0)
+			(at -1.814 0.564 0)
 			(unlocked yes)
 			(layer "F.SilkS")
@@
 	)
 	(via
+		(at 100.5 63.8)
+		(size 0.4)
+		(drill 0.2)
+		(layers "F.Cu" "B.Cu")
+		(free yes)
+		(net 1)
+	)
+	(via
 		(at 105 81.5)
 		(size 0.4)
@@
 	)
 	(via
+		(at 100.8 81.2)
+		(size 0.4)
+		(drill 0.2)
+		(layers "F.Cu" "B.Cu")
+		(free yes)
+		(net 1)
+	)
+	(via
 		(at 104.9375 82.038)
 		(size 0.4)
@@
 	)
 	(via
+		(at 101.5 81.2)
+		(size 0.4)
+		(drill 0.2)
+		(layers "F.Cu" "B.Cu")
+		(free yes)
+		(net 1)
+	)
+	(via
 		(at 102.362 64.008)
 		(size 0.4)
@@
 	)
 	(via
-		(at 98.5 61.722)
+		(at 99.5 61.75)
 		(size 0.4)
 		(drill 0.2)
@@
 	)
 	(via
+		(at 109.4 72)
+		(size 0.4)
+		(drill 0.2)
+		(layers "F.Cu" "B.Cu")
+		(free yes)
+		(net 1)
+	)
+	(via
 		(at 99 68.5)
 		(size 0.4)
@@
 	)
 	(via
+		(at 101.1 66.75)
+		(size 0.4)
+		(drill 0.2)
+		(layers "F.Cu" "B.Cu")
+		(free yes)
+		(net 1)
+	)
+	(via
 		(at 93.75 68.75)
 		(size 0.4)
@@
 	)
 	(via
-		(at 100.838 64.262)
+		(at 100.6 64.6)
 		(size 0.4)
 		(drill 0.2)
@@
 	)
 	(via
+		(at 98.8 66.8)
+		(size 0.4)
+		(drill 0.2)
+		(layers "F.Cu" "B.Cu")
+		(free yes)
+		(net 1)
+	)
+	(via
 		(at 103.759 68.58)
 		(size 0.4)
@@
 	)
 	(via
+		(at 98.75 62)
+		(size 0.4)
+		(drill 0.2)
+		(layers "F.Cu" "B.Cu")
+		(free yes)
+		(net 1)
+	)
+	(via
+		(at 101.1 65.75)
+		(size 0.4)
+		(drill 0.2)
+		(layers "F.Cu" "B.Cu")
+		(free yes)
+		(net 1)
+	)
+	(via
 		(at 92.71 75.692)
 		(size 0.4)
@@
 	)
 	(via
+		(at 101 67.8)
+		(size 0.4)
+		(drill 0.2)
+		(layers "F.Cu" "B.Cu")
+		(free yes)
+		(net 1)
+	)
+	(via
 		(at 107.75 68.5)
 		(size 0.4)
@@
 	)
 	(via
+		(at 98.8 64.8)
+		(size 0.4)
+		(drill 0.2)
+		(layers "F.Cu" "B.Cu")
+		(free yes)
+		(net 1)
+	)
+	(via
 		(at 92.964 69.596)
 		(size 0.4)
@@
 	)
 	(via
+		(at 98.8 65.75)
+		(size 0.4)
+		(drill 0.2)
+		(layers "F.Cu" "B.Cu")
+		(free yes)
+		(net 1)
+	)
+	(via
 		(at 97.18 70.51)
 		(size 0.4)
@@
 	)
 	(via
+		(at 105.8 76.1)
+		(size 0.4)
+		(drill 0.2)
+		(layers "F.Cu" "B.Cu")
+		(free yes)
+		(net 1)
+	)
+	(via
 		(at 99.026613 60.889266)
 		(size 0.4)
@@
 	)
 	(segment
-		(start 103.124 70.358)
-		(end 102.362 70.358)
+		(start 109.075 72.675)
+		(end 108.766 72.984)
 		(width 0.2)
 		(layer "F.Cu")
@@
 	)
 	(segment
-		(start 108.766 73.89)
-		(end 108.766 72.984)
+		(start 103.124 70.358)
+		(end 102.362 70.358)
 		(width 0.2)
 		(layer "F.Cu")
@@
 	(segment
 		(start 108.766 72.984)
-		(end 109.25 72.5)
+		(end 108.766 73.89)
 		(width 0.2)
 		(layer "F.Cu")
@@
 	)
 	(via
-		(at 109.25 72.5)
+		(at 109.075 72.675)
 		(size 0.4)
 		(drill 0.2)
@@
 	(segment
 		(start 106.718646 69.968646)
-		(end 109.25 72.5)
+		(end 103.513354 69.968646)
+		(width 0.2)
+		(layer "In1.Cu")
+		(net 26)
+	)
+	(segment
+		(start 109.075 72.675)
+		(end 108.8 72.4)
+		(width 0.2)
+		(layer "In1.Cu")
+		(net 26)
+	)
+	(segment
+		(start 108.8 72.4)
+		(end 108.8 72.05)
 		(width 0.2)
 		(layer "In1.Cu")
@@
 	(segment
 		(start 103.513354 69.968646)
-		(end 106.718646 69.968646)
+		(end 103.124 70.358)
 		(width 0.2)
 		(layer "In1.Cu")
@@
 	)
 	(segment
-		(start 103.124 70.358)
-		(end 103.513354 69.968646)
+		(start 108.8 72.05)
+		(end 106.718646 69.968646)
 		(width 0.2)
 		(layer "In1.Cu")
@@
 	)
 	(segment
-		(start 106 73)
-		(end 105.922 73.078)
+		(start 107.446523 76.846523)
+		(end 107.446523 78.786268)
 		(width 0.2)
 		(layer "In1.Cu")
@@
 	)
 	(segment
-		(start 107.446523 77.853523)
-		(end 107.446523 78.786268)
+		(start 106 73)
+		(end 105.922 73.078)
 		(width 0.2)
 		(layer "In1.Cu")
@@
 	(segment
 		(start 105.922 73.078)
-		(end 105.922 76.329)
+		(end 105.922 75.322)
 		(width 0.2)
 		(layer "In1.Cu")
@@
 	)
 	(segment
-		(start 105.922 76.329)
-		(end 107.446523 77.853523)
+		(start 105.922 75.322)
+		(end 107.446523 76.846523)
 		(width 0.2)
 		(layer "In1.Cu")

Commit message: Hardware V2 Finished
Parts:
- added TP1: TestPoint, TestPoint:TestPoint_Pad_D1.0mm, F.Cu at (97.9, 81.5)
- added TP10: TestPoint, TestPoint:TestPoint_Pad_D1.0mm, F.Cu at (94.7, 79.0)
- added TP11: TestPoint, TestPoint:TestPoint_Pad_D1.0mm, F.Cu at (94.2, 68.6)
- added TP2: TestPoint, TestPoint:TestPoint_Pad_D1.0mm, F.Cu at (112.3, 78.0)
- added TP4: TestPoint, TestPoint:TestPoint_Pad_D1.0mm, F.Cu at (106.3, 70.1)
- added TP5: TestPoint, TestPoint:TestPoint_Pad_D1.0mm, F.Cu at (104.4, 70.1)
- added TP6: TestPoint, TestPoint:TestPoint_Pad_D1.0mm, F.Cu at (105.2, 75.6)
- added TP7: TestPoint, TestPoint:TestPoint_Pad_D1.0mm, F.Cu at (106.4, 67.4)
- added TP8: TestPoint, TestPoint:TestPoint_Pad_D1.0mm, F.Cu at (108.1, 69.1)
- added TP9: TestPoint, TestPoint:TestPoint_Pad_D1.0mm, F.Cu at (112.3, 69.1)
- moved R3 0.10 mm to (104.9, 67.2)
- moved C30 0.09 mm to (102.2, 67.8)
- moved R6 0.09 mm to (103.7, 78.3)
Connections:
- C26 pad 1: +1V8 -> GND
- U4 pad 33: (no net) -> GND
Routing:
- net +1V8: track 87.6 -> 92.4 mm, vias 8 -> 16
- net /IMU_INT: track 8.99 -> 13.0 mm
- net /UART_TX: track 17.6 -> 20.6 mm
- net /SW_IMU: track 9.80 -> 12.6 mm
- net /MISO: track 10.5 -> 13.2 mm, vias 2 -> 3
- net /LED: track 10.1 -> 7.49 mm
- net /~{SS}: track 8.80 -> 10.6 mm
- net /MOSI: track 9.57 -> 11.1 mm
- net /BATT_EN: track 11.1 -> 10.1 mm
- net +BATT: track 22.2 -> 23.3 mm, vias 1 -> 2
- net GND: track 37.1 -> 37.3 mm, vias 118 -> 145
Other:
- board text added: "CR2032"
- board text added: "KUL Logo"
- board text added: "W"
- board text added: "e"
